File: hardware/portfire.kicad_pcb (KiCad board)
At the start: 2 copper layers, 100 x 100 mm, 31 parts, among them P101 1, P102 11, P103 2, P104 12, P105 3, P106 13, P107 4, P108 14, P109 5, P110 15, P111 6, P112 21, P113 7, P114 22, P115 8, P116 23, P117 9, P118 24, P119 10, P120 25, P121 16, P122 17, P123 18, P124 19, P125 20, P126 26, P127 27, P128 28, P129 29, P130 30

Commit message: Fixed fp references
Parts:
- removed J?: RJ45, Connect:RJ45_8
- removed P101: 1, hardware:PTSA0,52-2,5-z
- removed P102: 11, hardware:PTSA0,52-2,5-z
- removed P103: 2, hardware:PTSA0,52-2,5-z
- removed P104: 12, hardware:PTSA0,52-2,5-z
- removed P105: 3, hardware:PTSA0,52-2,5-z
- removed P106: 13, hardware:PTSA0,52-2,5-z
- removed P107: 4, hardware:PTSA0,52-2,5-z
- removed P108: 14, hardware:PTSA0,52-2,5-z
- removed P109: 5, hardware:PTSA0,52-2,5-z
- removed P110: 15, hardware:PTSA0,52-2,5-z
- removed P111: 6, hardware:PTSA0,52-2,5-z
- removed P112: 21, hardware:PTSA0,52-2,5-z
- removed P113: 7, hardware:PTSA0,52-2,5-z
- removed P114: 22, hardware:PTSA0,52-2,5-z
- removed P115: 8, hardware:PTSA0,52-2,5-z
- removed P116: 23, hardware:PTSA0,52-2,5-z
- removed P117: 9, hardware:PTSA0,52-2,5-z
- removed P118: 24, hardware:PTSA0,52-2,5-z
- removed P119: 10, hardware:PTSA0,52-2,5-z
- removed P120: 25, hardware:PTSA0,52-2,5-z
- removed P121: 16, hardware:PTSA0,52-2,5-z
- removed P122: 17, hardware:PTSA0,52-2,5-z
- removed P123: 18, hardware:PTSA0,52-2,5-z
- removed P124: 19, hardware:PTSA0,52-2,5-z
- removed P125: 20, hardware:PTSA0,52-2,5-z
- removed P126: 26, hardware:PTSA0,52-2,5-z
- removed P127: 27, hardware:PTSA0,52-2,5-z
- removed P128: 28, hardware:PTSA0,52-2,5-z
- removed P129: 29, hardware:PTSA0,52-2,5-z
- removed P130: 30, hardware:PTSA0,52-2,5-z
- added C1: 2u2 60V, agg:1210, F.Cu at (241.2, 121.4)
- added C10: 100n, agg:0603, F.Cu at (271.6, 112.0)
- added C11: 2u2, agg:0603, F.Cu at (255.0, 122.8)
- added C12: 100n, agg:0603, F.Cu at (262.5, 116.5)
- added C13: 22u, agg:1206, F.Cu at (267.3, 96.9)
- added C14: 22u, agg:1206, F.Cu at (257.4, 105.0)
- added C2: 10n 200V, agg:0805, F.Cu at (257.4, 110.5)
- added C3: 18n 50V, agg:0603, F.Cu at (256.0, 117.7)
- added C4: 10n 200V, agg:0805, F.Cu at (184.2, 117.7)
- added C5: 1n 2kV, agg:1206, F.Cu at (249.9, 110.4)
- added C6: 10n 200V, agg:0805, F.Cu at (249.3, 117.0)
- added C7: 10n 200V, agg:0805, F.Cu at (274.8, 98.5)
- added C8: 100n 60V, agg:0805, F.Cu at (264.9, 109.3)
- added C9: 100n, agg:0603, F.Cu at (261.5, 123.2)
- added D1: SS110B, agg:DO-214AA-SMB, F.Cu at (231.8, 120.3)
- added D2: SS110B, agg:DO-214AA-SMB, F.Cu at (247.9, 104.5)
- added D3: SS110B, agg:DO-214AA-SMB, F.Cu at (247.9, 98.3)
- added D4: SS110B, agg:DO-214AA-SMB, F.Cu at (231.8, 114.1)
- added D5: SS110B, agg:DO-214AA-SMB, F.Cu at (221.0, 120.3)
- added D6: SS110B, agg:DO-214AA-SMB, F.Cu at (221.0, 114.1)
- added D7: SS110B, agg:DO-214AA-SMB, F.Cu at (210.3, 120.3)
- added D8: SS110B, agg:DO-214AA-SMB, F.Cu at (210.3, 114.1)
- added D9: SMAJ58A, agg:DO-214AC-SMA, F.Cu at (273.0, 82.9)
- added IC1: MAX17503, agg:QFN-20-EP-MAX, F.Cu at (271.9, 90.4)
- added IC2: MAX5969x, agg:DFN-10-EP-MAX, F.Cu at (267.3, 102.0)
- added IC3: KSZ8081RNx, agg:QFN-24-EP-MICREL, F.Cu at (258.3, 99.3)
- added IC4: 25AA02E48, agg:SOT-23-6, F.Cu at (241.6, 114.5)
- added IC5: STM32F4xxVxTx, agg:LQFP-100, F.Cu at (178.1, 97.1)
- added J1: RJ45, Connect:RJ45_8, F.Cu at (190.4, 74.0)
- added L1: 3u3, hardware:ELLATP3R3NB, F.Cu at (199.5, 116.6)
- added L2: SRR1260A-120M, hardware:SRR1260A, F.Cu at (175.8, 70.1)
- added P1: 1, hardware:PTSA0,52-2,5-z, F.Cu at (202.5, 68.7)
- added P10: 10, hardware:PTSA0,52-2,5-z, F.Cu at (251.2, 84.5)
- added P11: 11, hardware:PTSA0,52-2,5-z, F.Cu at (232.9, 100.3)
- added P12: 12, hardware:PTSA0,52-2,5-z, F.Cu at (265.1, 68.7)
- added P13: 13, hardware:PTSA0,52-2,5-z, F.Cu at (258.1, 68.7)
- added P14: 14, hardware:PTSA0,52-2,5-z, F.Cu at (244.2, 84.5)
- added P15: 15, hardware:PTSA0,52-2,5-z, F.Cu at (225.9, 100.3)
- added P16: 16, hardware:PTSA0,52-2,5-z, F.Cu at (237.3, 84.5)
- added P17: 17, hardware:PTSA0,52-2,5-z, F.Cu at (251.2, 68.7)
- added P18: 18, hardware:PTSA0,52-2,5-z, F.Cu at (219.0, 100.3)
- added P19: 19, hardware:PTSA0,52-2,5-z, F.Cu at (212.0, 100.3)
- added P2: 2, hardware:PTSA0,52-2,5-z, F.Cu at (191.2, 103.1)
- added P20: 20, hardware:PTSA0,52-2,5-z, F.Cu at (244.2, 68.7)
- added P21: 21, hardware:PTSA0,52-2,5-z, F.Cu at (230.3, 84.5)
- added P22: 22, hardware:PTSA0,52-2,5-z, F.Cu at (237.3, 68.7)
- added P23: 23, hardware:PTSA0,52-2,5-z, F.Cu at (216.4, 84.5)
- added P24: 24, hardware:PTSA0,52-2,5-z, F.Cu at (209.5, 84.5)
- added P25: 25, hardware:PTSA0,52-2,5-z, F.Cu at (202.5, 84.5)
- added P26: 26, hardware:PTSA0,52-2,5-z, F.Cu at (230.3, 68.7)
- added P27: 27, hardware:PTSA0,52-2,5-z, F.Cu at (223.4, 68.7)
- added P28: 28, hardware:PTSA0,52-2,5-z, F.Cu at (216.4, 68.7)
- added P29: 29, hardware:PTSA0,52-2,5-z, F.Cu at (209.5, 68.7)
- added P3: 3, hardware:PTSA0,52-2,5-z, F.Cu at (198.1, 100.3)
- added P30: 30, hardware:PTSA0,52-2,5-z, F.Cu at (191.2, 87.3)
- added P4: 4, hardware:PTSA0,52-2,5-z, F.Cu at (223.4, 84.5)
- added P5: 5, hardware:PTSA0,52-2,5-z, F.Cu at (205.1, 100.3)
- added P6: 6, hardware:PTSA0,52-2,5-z, F.Cu at (265.1, 84.5)
- added P7: 7, hardware:PTSA0,52-2,5-z, F.Cu at (258.1, 84.5)
- added P8: 8, hardware:PTSA0,52-2,5-z, F.Cu at (272.0, 68.7)
- added P9: 9, hardware:PTSA0,52-2,5-z, F.Cu at (239.8, 100.3)
- added R1: 75, agg:0603, F.Cu at (227.7, 124.6)
- added R2: 75, agg:0603, F.Cu at (221.2, 124.6)
- added R3: 3M3, agg:0603, F.Cu at (271.6, 108.2)
- added R4: 75, agg:0603, F.Cu at (214.7, 124.6)
- added R5: 75, agg:0603, F.Cu at (208.2, 124.6)
- added R6: 24k9, agg:0603, F.Cu at (274.5, 104.4)
- added R7: 619, agg:0603, F.Cu at (248.5, 122.5)
- added R8: 88k7, agg:0603, F.Cu at (190.5, 123.5)
- added R9: 15k8, agg:0603, F.Cu at (184.0, 123.5)
- added T1: 749010012A, agg:749010012A, F.Cu at (175.0, 115.8)
Other:
- board outline removed
- net class Default: via_dia 0.8 -> 0.6
- rule pad_to_mask_clearance: 0.2 -> 0

Commit message: Firing matrix and CC SMPS
Parts:
- removed C1: 2u2 60V, agg:1210
- removed C10, C12, C9: 100n, agg:0603
- removed C11: 2u2, agg:0603
- removed C13, C14: 22u, agg:1206
- removed C2, C4, C6, C7: 10n 200V, agg:0805
- removed C3: 18n 50V, agg:0603
- removed C5: 1n 2kV, agg:1206
- removed C8: 100n 60V, agg:0805
- removed D1, D2, D3, D4, D5, D6, D7, D8: SS110B, agg:DO-214AA-SMB
- removed D9: SMAJ58A, agg:DO-214AC-SMA
- removed IC1: MAX17503, agg:QFN-20-EP-MAX
- removed IC2: MAX5969x, agg:DFN-10-EP-MAX
- removed IC3: KSZ8081RNx, agg:QFN-24-EP-MICREL
- removed IC4: 25AA02E48, agg:SOT-23-6
- removed IC5: STM32F4xxVxTx, agg:LQFP-100
- removed J1: RJ45, Connect:RJ45_8
- removed L1: 3u3, hardware:ELLATP3R3NB
- removed L2: SRR1260A-120M, hardware:SRR1260A
- removed P1: 1, hardware:PTSA0,52-2,5-z
- removed P10: 10, hardware:PTSA0,52-2,5-z
- removed P11: 11, hardware:PTSA0,52-2,5-z
- removed P12: 12, hardware:PTSA0,52-2,5-z
- removed P13: 13, hardware:PTSA0,52-2,5-z
- removed P14: 14, hardware:PTSA0,52-2,5-z
- removed P15: 15, hardware:PTSA0,52-2,5-z
- removed P16: 16, hardware:PTSA0,52-2,5-z
- removed P17: 17, hardware:PTSA0,52-2,5-z
- removed P18: 18, hardware:PTSA0,52-2,5-z
- removed P19: 19, hardware:PTSA0,52-2,5-z
- removed P2: 2, hardware:PTSA0,52-2,5-z
- removed P20: 20, hardware:PTSA0,52-2,5-z
- removed P21: 21, hardware:PTSA0,52-2,5-z
- removed P22: 22, hardware:PTSA0,52-2,5-z
- removed P23: 23, hardware:PTSA0,52-2,5-z
- removed P24: 24, hardware:PTSA0,52-2,5-z
- removed P25: 25, hardware:PTSA0,52-2,5-z
- removed P26: 26, hardware:PTSA0,52-2,5-z
- removed P27: 27, hardware:PTSA0,52-2,5-z
- removed P28: 28, hardware:PTSA0,52-2,5-z
- removed P29: 29, hardware:PTSA0,52-2,5-z
- removed P3: 3, hardware:PTSA0,52-2,5-z
- removed P30: 30, hardware:PTSA0,52-2,5-z
- removed P4: 4, hardware:PTSA0,52-2,5-z
- removed P5: 5, hardware:PTSA0,52-2,5-z
- removed P6: 6, hardware:PTSA0,52-2,5-z
- removed P7: 7, hardware:PTSA0,52-2,5-z
- removed P8: 8, hardware:PTSA0,52-2,5-z
- removed P9: 9, hardware:PTSA0,52-2,5-z
- removed R1, R2, R4, R5: 75, agg:0603
- removed R3: 3M3, agg:0603
- removed R6: 24k9, agg:0603
- removed R7: 619, agg:0603
- removed R8: 88k7, agg:0603
- removed R9: 15k8, agg:0603
- removed T1: 749010012A, agg:749010012A
- added C101: 100n, agg:0603, F.Cu at (262.9, 21.4)
- added C102: 2u2, agg:0603, F.Cu at (248.5, 33.0)
- added C103: 2u2, agg:0603, F.Cu at (248.5, 28.7)
- added C104: 100n, agg:0603, F.Cu at (256.4, 21.4)
- added C105: 100n, agg:0603, F.Cu at (264.7, 17.1)
- added C106: 1u, agg:0603, F.Cu at (256.4, 25.6)
- added C107: 4u7, agg:0603, F.Cu at (246.8, 38.0)
- added C108: 100n, agg:0603, F.Cu at (271.2, 17.1)
- added C109: 100n, agg:0603, F.Cu at (255.0, 29.9)
- added C110: 100n, agg:0603, F.Cu at (262.9, 25.6)
- added C111: 100n, agg:0603, F.Cu at (269.4, 21.4)
- added C112: 100n, agg:0603, F.Cu at (255.0, 34.1)
- added C113: 100n, agg:0603, F.Cu at (261.5, 29.9)
- added C114: 22u, agg:1206, F.Cu at (257.4, 17.1)
- added C115: 100n, agg:0603, F.Cu at (253.3, 38.4)
- added C116: 3n3, agg:0603, F.Cu at (269.4, 25.6)
- added C117: 22u, agg:1206, F.Cu at (249.3, 17.1)
- added C201: 10n 200V, agg:0805, F.Cu at (153.1, 109.6)
- added C202: 10n 200V, agg:0805, F.Cu at (142.4, 122.0)
- added C203: 1n 2kV, agg:1206, F.Cu at (145.6, 111.5)
- added C204: 10n 200V, agg:0805, F.Cu at (134.3, 128.4)
- added C205: 10n 200V, agg:0805, F.Cu at (173.9, 89.1)
- added C206: 100n 60V, agg:0805, F.Cu at (154.7, 102.0)
- added C207: 100n, agg:0603, F.Cu at (152.9, 115.6)
- added C208: 100n, agg:0603, F.Cu at (141.0, 128.0)
- added C209: 2u2, agg:0603, F.Cu at (149.1, 119.8)
- added C210: 100n, agg:0603, F.Cu at (162.1, 119.8)
- added C211: 30p, agg:0603, F.Cu at (165.9, 115.2)
- added C212: 2u2 60V, agg:1210, F.Cu at (155.6, 94.7)
- added C213: 30p, agg:0603, F.Cu at (155.6, 124.1)
- added C214: 22u, agg:1206, F.Cu at (166.4, 87.3)
- added C215: 18n 50V, agg:0603, F.Cu at (170.9, 96.3)
- added C216: 100n, agg:0603, F.Cu at (183.9, 95.8)
- added C217: 22u, agg:1206, F.Cu at (134.9, 122.5)
- added C218: 100n, agg:0603, F.Cu at (174.4, 106.0)
- added C219: 2u2, agg:0603, F.Cu at (161.4, 106.7)
- added C220: 100n, agg:0603, F.Cu at (180.6, 87.3)
- added C221: 10u, agg:0603, F.Cu at (127.0, 130.6)
- added C222: 22u, agg:1206, F.Cu at (145.6, 106.5)
- added C223: 22u, agg:1206, F.Cu at (119.8, 130.6)
- added C301: 22u, agg:1206, F.Cu at (154.5, 78.5)
- added C302: 10n, agg:0805, F.Cu at (108.4, 71.9)
- added C303: 100n, agg:0603, F.Cu at (210.8, 49.2)
- added C304: 100n, agg:0603, F.Cu at (186.1, 71.9)
- added C305: 4u7, agg:0603, F.Cu at (186.1, 67.7)
- added D201: SS110B, agg:DO-214AA-SMB, F.Cu at (123.6, 105.0)
- added D202: SS110B, agg:DO-214AA-SMB, F.Cu at (135.2, 101.4)
- added D203: SS110B, agg:DO-214AA-SMB, F.Cu at (146.2, 88.3)
- added D204: SS110B, agg:DO-214AA-SMB, F.Cu at (110.3, 130.0)
- added D205: SS110B, agg:DO-214AA-SMB, F.Cu at (126.2, 111.1)
- added D206: SS110B, agg:DO-214AA-SMB, F.Cu at (126.2, 117.3)
- added D207: SS110B, agg:DO-214AA-SMB, F.Cu at (156.9, 88.3)
- added D208: SS110B, agg:DO-214AA-SMB, F.Cu at (146.2, 94.5)
- added D209: SMAJ58A, agg:DO-214AC-SMA, F.Cu at (146.0, 101.0)
- added D210: 1N4148, agg:SOD-323, F.Cu at (161.9, 101.4)
- added D301: PMEG2005AEA, agg:SOD-323, F.Cu at (191.2, 20.4)
- added D302: PMEG2005AEA, agg:SOD-323, F.Cu at (143.4, 67.9)
- added D303: SS110B, agg:DO-214AA-SMB, F.Cu at (177.4, 77.5)
- added D304: STPS3L40UF, agg:DO-214AA-SMB, F.Cu at (202.1, 54.6)
- added IC101: STM32F4xxVxTx, agg:LQFP-100, F.Cu at (236.4, 25.4)
- added IC102: TPS62152, agg:QFN-16-EP-TI, F.Cu at (249.2, 22.9)
- added IC103: 25AA02E48, agg:SOT-23-6, F.Cu at (231.8, 39.3)
- added IC201: MAX5969x, agg:DFN-10-EP-MAX, F.Cu at (163.7, 94.8)
- added IC202: KSZ8081RNA, agg:QFN-24-EP-MICREL, F.Cu at (125.9, 124.4)
- added IC203: MAX17503, agg:QFN-20-EP-MAX, F.Cu at (135.7, 113.9)
- added J201: RJ45, Connect:RJ45_8, F.Cu at (113.0, 118.8)
- added L101: 3u3, agg:VLS201610HBX-1, F.Cu at (261.2, 34.0)
- added L201: 3u3, hardware:ELLATP3R3NB, F.Cu at (135.4, 90.7)
- added L202: FB, agg:0603, F.Cu at (168.9, 101.7)
- added L203: SRR1260A-120M, hardware:SRR1260A, F.Cu at (111.6, 91.7)
- added L301: 12uH, hardware:SRR1260A, F.Cu at (111.5, 21.5)
- added P101: SWD_TC, agg:TC2030-NL, F.Cu at (239.9, 39.4)
- added P301: 1, hardware:PTSA0,52-2,5-z, F.Cu at (170.9, 20.1)
- added P302: 2, hardware:PTSA0,52-2,5-z, F.Cu at (157.0, 35.9)
- added P303: 3, hardware:PTSA0,52-2,5-z, F.Cu at (163.9, 20.1)
- added P304: 4, hardware:PTSA0,52-2,5-z, F.Cu at (150.0, 35.9)
- added P305: 5, hardware:PTSA0,52-2,5-z, F.Cu at (116.1, 67.5)
- added P306: 6, hardware:PTSA0,52-2,5-z, F.Cu at (130.0, 51.7)
- added P307: 7, hardware:PTSA0,52-2,5-z, F.Cu at (123.1, 51.7)
- added P308: 8, hardware:PTSA0,52-2,5-z, F.Cu at (116.1, 51.7)
- added P309: 9, hardware:PTSA0,52-2,5-z, F.Cu at (143.1, 35.9)
- added P310: 10, hardware:PTSA0,52-2,5-z, F.Cu at (136.1, 35.9)
- added P311: 11, hardware:PTSA0,52-2,5-z, F.Cu at (129.2, 35.9)
- added P312: 12, hardware:PTSA0,52-2,5-z, F.Cu at (157.0, 20.1)
- added P313: 13, hardware:PTSA0,52-2,5-z, F.Cu at (150.0, 20.1)
- added P314: 14, hardware:PTSA0,52-2,5-z, F.Cu at (143.1, 20.1)
- added P315: 15, hardware:PTSA0,52-2,5-z, F.Cu at (136.1, 20.1)
- added P316: 16, hardware:PTSA0,52-2,5-z, F.Cu at (122.2, 35.9)
- added P317: 17, hardware:PTSA0,52-2,5-z, F.Cu at (129.2, 20.1)
- added P318: 18, hardware:PTSA0,52-2,5-z, F.Cu at (109.2, 59.0)
- added P319: 19, hardware:PTSA0,52-2,5-z, F.Cu at (122.2, 20.1)
- added P320: 20, hardware:PTSA0,52-2,5-z, F.Cu at (109.2, 43.2)
- added P321: 21, hardware:PTSA0,52-2,5-z, F.Cu at (137.0, 67.5)
- added P322: 22, hardware:PTSA0,52-2,5-z, F.Cu at (184.8, 20.1)
- added P323: 23, hardware:PTSA0,52-2,5-z, F.Cu at (170.9, 35.9)
- added P324: 24, hardware:PTSA0,52-2,5-z, F.Cu at (150.9, 51.7)
- added P325: 25, hardware:PTSA0,52-2,5-z, F.Cu at (163.9, 35.9)
- added P326: 26, hardware:PTSA0,52-2,5-z, F.Cu at (177.8, 20.1)
- added P327: 27, hardware:PTSA0,52-2,5-z, F.Cu at (143.9, 51.7)
- added P328: 28, hardware:PTSA0,52-2,5-z, F.Cu at (130.0, 67.5)
- added P329: 29, hardware:PTSA0,52-2,5-z, F.Cu at (137.0, 51.7)
- added P330: 30, hardware:PTSA0,52-2,5-z, F.Cu at (123.1, 67.5)
- added Q301: NTR4501NT1G, agg:SOT-23, F.Cu at (189.8, 36.2)
- added Q302: NTR4501NT1G, agg:SOT-23, F.Cu at (180.6, 48.1)
- added Q303: NTR4501NT1G, agg:SOT-23, F.Cu at (169.8, 57.0)
- added Q304: NTR4501NT1G, agg:SOT-23, F.Cu at (192.9, 29.3)
- added Q305: NTR4501NT1G, agg:SOT-23, F.Cu at (145.1, 76.8)
- added Q306: NTR4501NT1G, agg:SOT-23, F.Cu at (152.6, 65.9)
- added Q307: NTR4501NT1G, agg:SOT-23, F.Cu at (200.4, 18.4)
- added Q308: NTR4501NT1G, agg:SOT-23, F.Cu at (179.0, 41.2)
- added Q309: NTR4501NT1G, agg:SOT-23, F.Cu at (169.8, 50.1)
- added Q310: NTR4501NT1G, agg:SOT-23, F.Cu at (159.0, 57.0)
- added Q311: NTR4501NT1G, agg:SOT-23, F.Cu at (179.0, 34.2)
- added Q312: NTR4501NT1G, agg:SOT-23, F.Cu at (177.5, 70.9)
- added Q313: NTR4501NT1G, agg:SOT-23, F.Cu at (202.2, 46.2)
- added Q314: NTR4501NT1G, agg:SOT-23, F.Cu at (184.9, 62.0)
- added Q315: NTR4501NT1G, agg:SOT-23, F.Cu at (214.5, 32.3)
- added Q316: NTR4501NT1G, agg:SOT-23, F.Cu at (202.2, 39.3)
- added Q317: NTR4501NT1G, agg:SOT-23, F.Cu at (166.7, 77.9)
- added Q318: NTR4501NT1G, agg:SOT-23, F.Cu at (191.4, 50.1)
- added Q319: NTR4501NT1G, agg:SOT-23, F.Cu at (159.0, 50.1)
- added Q320: NTR4501NT1G, agg:SOT-23, F.Cu at (163.4, 64.0)
- added Q321: NTR4501NT1G, agg:SOT-23, F.Cu at (211.2, 18.4)
- added Q322: NTR4501NT1G, agg:SOT-23, F.Cu at (155.9, 72.8)
- added Q323: NTR4501NT1G, agg:SOT-23, F.Cu at (203.7, 25.4)
- added Q324: NTR4501NT1G, agg:SOT-23, F.Cu at (180.6, 55.1)
- added Q325: NTR4501NT1G, agg:SOT-23, F.Cu at (203.7, 32.3)
- added Q326: NTR4501NT1G, agg:SOT-23, F.Cu at (191.4, 43.2)
- added Q327: NTR4501NT1G, agg:SOT-23, F.Cu at (174.2, 64.0)
- added Q328: NTR4501NT1G, agg:SOT-23, F.Cu at (214.5, 25.4)
- added Q329: NTR4501NT1G, agg:SOT-23, F.Cu at (166.7, 70.9)
- added Q330: NTR4501NT1G, agg:SOT-23, F.Cu at (212.9, 39.3)
- added R201: 75, agg:0603, F.Cu at (180.6, 91.6)
- added R202: 75, agg:0603, F.Cu at (159.8, 110.9)
- added R203: 75, agg:0603, F.Cu at (167.9, 106.7)
- added R204: 75, agg:0603, F.Cu at (149.1, 124.1)
- added R205: 24k9, agg:0603, F.Cu at (187.1, 87.3)
- added R206: 619, agg:0603, F.Cu at (159.4, 115.6)
- added R207: 3M3, agg:0603, F.Cu at (155.6, 119.8)
- added R208: 6k49, agg:0603, F.Cu at (175.4, 101.8)
- added R209: 1k, agg:0603, F.Cu at (177.4, 95.8)
- added R210: 10k, agg:0603, F.Cu at (187.1, 91.6)
- added R211: 88k7, agg:0603, F.Cu at (147.5, 128.3)
- added R212: 15k8, agg:0603, F.Cu at (166.3, 110.9)
- added R301: 30k, agg:0603, F.Cu at (210.8, 44.9)
- added R302: 10k, agg:0603, F.Cu at (189.2, 55.8)
- added R303: 10M, agg:0603, F.Cu at (219.8, 17.1)
- added R304: 3k3, agg:0603, F.Cu at (108.2, 76.1)
- added R305: 200k, agg:0603, F.Cu at (193.5, 61.5)
- added R306: 3k3, agg:0603, F.Cu at (193.5, 65.8)
- added R307: 1k, agg:0603, F.Cu at (200.0, 61.5)
- added T201: 749010012A, agg:749010012A, F.Cu at (124.1, 93.5)
- added Y201: 25MHz, agg:XTAL-50x32, F.Cu at (136.6, 107.1)

Commit message: aux power, test points
Parts:
- added J202: AUX POWER, hardware:Minipow, F.Cu at (149.9, 34.9)
- added JP201: Jumper_NC_Small, hardware:jump_NC, F.Cu at (175.2, -6.42)
- added R308: 0R15 1W, agg:2512, F.Cu at (60.4, 41.0)
- added TP101: 3v3, hardware:Test_point_mini, F.Cu at (67.7, 67.4)
- added TP201: +48V, hardware:Test_point_mini, F.Cu at (228.3, 7.08)
- added TP202: DCDC_EN, hardware:Test_point_mini, F.Cu at (181.3, 36.1)
- added TP203: 25MHz_XTAL, agg:TESTPAD, F.Cu at (194.3, 0.53)
- added TP204: 50MHz_CLK, agg:TESTPAD, F.Cu at (173.5, 28.3)
- added TP205: 6V_SMPS, hardware:Test_point_mini, F.Cu at (199.4, 17.4)
- added TP206: 6V_BUS, hardware:Test_point_mini, F.Cu at (211.9, 25.7)
- added TP301: CONT_EN, agg:TESTPAD, F.Cu at (135.0, -7.62)
- added TP302: ARM, agg:TESTPAD, F.Cu at (137.4, -2.58)
- added TP303: CONT_MEAS, agg:TESTPAD, F.Cu at (59.2, 53.9)
- added TP304: BUS, hardware:Test_point_mini, F.Cu at (29.5, 15.7)
- added TP305: RETURN, hardware:Test_point_mini, F.Cu at (114.9, 34.3)
- moved C110 227.1 mm to (41.0, 74.3)
- moved C106 224.6 mm to (39.3, 83.6)
- moved C101 223.1 mm to (47.5, 79.7)
- moved C111 218.8 mm to (55.4, 67.0)
- moved C108 218.8 mm to (57.2, 62.7)
- moved C104 215.7 mm to (47.5, 75.5)
- moved C113 212.4 mm to (54.0, 75.5)
- moved C116 212.4 mm to (61.9, 71.2)
- moved C114 212.4 mm to (49.9, 62.7)
- moved C115 212.4 mm to (45.8, 84.0)
- moved C117 212.4 mm to (41.8, 62.7)
- moved IC101 212.4 mm to (28.9, 71.0)
- moved IC102 212.4 mm to (41.7, 68.5)
- moved IC103 212.4 mm to (24.4, 84.9)
- moved P101 212.4 mm to (32.4, 85.0)
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Connections:
- C222 pad 1: +6V -> Net-(C222-Pad1)
- C223 pad 1: +6V -> Net-(C222-Pad1)
- L203 pad 1: +6V -> Net-(C222-Pad1)
- R211 pad 1: +6V -> Net-(C222-Pad1)

Commit message: Added aux bus
Parts:
- added C118: 2u2, agg:0603, F.Cu at (297.7, 88.1)
- added C119: 100n, agg:0603, F.Cu at (312.9, 70.6)
- added C120: 2u2, agg:0603, F.Cu at (306.4, 78.0)
- added IC104: ADP3335, agg:MSOP-8, F.Cu at (285.1, 79.7)
- added IC105: SNx5176B, agg:SOIC-8, F.Cu at (295.2, 64.4)
- added IC301: TPS92512, agg:MSOP-10-EP-TI, F.Cu at (246.5, 91.2)
- added P102: AUX_BUS_RX, agg:B02B-PASK, F.Cu at (286.4, 64.6)
- added P103: AUX_BUS_RX, agg:B02B-PASK, F.Cu at (268.6, 85.4)
- moved P101 271.4 mm to (302.9, 63.6)
- moved C101 269.2 mm to (316.4, 66.4)
- moved C107 269.1 mm to (309.9, 66.4)
- moved C110 269.1 mm to (309.9, 62.1)
- moved IC103 261.8 mm to (285.9, 72.7)
- moved L101 259.0 mm to (312.7, 74.8)
- moved C117 253.6 mm to (295.2, 71.1)
- moved C105 252.6 mm to (316.4, 62.1)
- moved C106 252.4 mm to (291.8, 83.8)
- moved C109 251.2 mm to (299.9, 75.3)
- moved C103 251.1 mm to (306.4, 73.8)
- moved C104 250.8 mm to (298.3, 79.6)
- moved C113 248.6 mm to (302.5, 69.5)
- moved C115 247.7 mm to (293.4, 75.3)
- moved IC101 243.7 mm to (272.6, 70.4)
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Connections:
- C303 pad 1: (no net) -> Net-(C303-Pad1)
- C304 pad 1: (no net) -> Net-(C304-Pad1)
- R305 pad 1: (no net) -> Net-(IC301-Pad5)
- R307 pad 2: (no net) -> Net-(IC301-Pad7)
- TP302 pad 1: (no net) -> /firing/ARM
