File: hardware/firing.sch (KiCad schematic (older format))
At the start: 84 parts, among them IC301 TPS92512, P301 1, P302 2, P303 3, P304 4, P305 5, P306 6, P307 7, P308 8, P309 9, P310 10, P311 11, P312 12, P313 13, P314 14, P315 15, P316 16, P317 17, P318 18, P319 19, P320 20, P321 21, P322 22, P323 23, P324 24, P325 25, P326 26, P327 27, P328 28, P329 29, P330 30, Q301 NTR4501NT1G, Q302 NTR4501NT1G, Q303 NTR4501NT1G, Q304 NTR4501NT1G, Q305 NTR4501NT1G, Q306 NTR4501NT1G, Q307 NTR4501NT1G, Q308 NTR4501NT1G, Q309 NTR4501NT1G, Q310 NTR4501NT1G, Q311 NTR4501NT1G, Q312 NTR4501NT1G, Q313 NTR4501NT1G, Q314 NTR4501NT1G, Q315 NTR4501NT1G, Q316 NTR4501NT1G, Q317 NTR4501NT1G, Q318 NTR4501NT1G, Q319 NTR4501NT1G, Q320 NTR4501NT1G, Q321 NTR4501NT1G, Q322 NTR4501NT1G, Q323 NTR4501NT1G, Q324 NTR4501NT1G, Q325 NTR4501NT1G, Q326 NTR4501NT1G, Q327 NTR4501NT1G, Q328 NTR4501NT1G, Q329 NTR4501NT1G, Q330 NTR4501NT1G

Commit message: Lots of placement/routing
Parts:
- removed TP304: BUS, hardware:Test_point_mini, symbol TESTPAD
- removed TP305: RETURN, hardware:Test_point_mini, symbol TESTPAD
Changed lines of the file:
@@
 Text Label 3850 6600 2    60   ~ 0
 RETURN
-$Comp
-L TESTPAD TP304
-U 1 1 57F3CEA9
-P 10200 4700
-F 0 "TP304" H 10200 4750 50  0000 L CNN
-F 1 "BUS" H 10200 4625 50  0001 L CNN
-F 2 "hardware:Test_point_mini" H 10200 4550 50  0001 L CNN
-F 3 "" H 10200 4700 50  0001 C CNN
-	1    10200 4700
-	0    -1   -1   0
-$EndComp
-Wire Wire Line
-	10200 4700 10200 4750
-Connection ~ 10200 4750
-$Comp
-L TESTPAD TP305
-U 1 1 57F3DDB8
-P 10200 4950
-F 0 "TP305" H 10200 5000 50  0000 L CNN
-F 1 "RETURN" H 10200 4875 50  0001 L CNN
-F 2 "hardware:Test_point_mini" H 10200 4800 50  0001 L CNN
-F 3 "" H 10200 4950 50  0001 C CNN
-	1    10200 4950
-	0    -1   -1   0
-$EndComp
 Wire Wire Line
 	10000 5000 10450 5000
-Connection ~ 10200 5000
-Wire Wire Line
-	10200 4950 10200 5000
 Wire Wire Line
 	7300 5050 7550 5050
